File: VoltageMeter/VoltageMeter.kicad_pcb (KiCad board)
At the start: 2 copper layers, 95.2 x 78.7 mm, 21 parts, among them J1 Conn_01x02_Male, J2 Conn_01x02_Male

Commit message: A few updates to clean things up.
Parts:
- TR2: footprint Transformer_THT:4900-XXXXRA60 -> VoltageMeter:4900-XXXXRA60
- moved REF5 1.65 mm to (71.0, 108.8)
Routing:
- net GND: track 77.3 -> 82.0 mm
Changed lines of the file:
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@@
 		)
 	)
-	(footprint "Transformer_THT:4900-XXXXRA60"
+	(footprint "VoltageMeter:4900-XXXXRA60"
 		(layer "F.Cu")
 		(at 110.003 145.875 -90)
@@
 			)
 		)
-		(property "Footprint" ""
+		(property "Footprint" "VoltageMeter:4900-XXXXRA60"
 			(at 0 0 90)
 			(layer "F.Fab")
@@
 		(pad "1" thru_hole rect
 			(at 8.03 31 270)
-			(size 2.286 2.286)
-			(drill 1.27)
+			(size 2.8 2.8)
+			(drill 1.5)
 			(layers "*.Cu" "*.Mask")
 			(remove_unused_layers no)
@@
 		(pad "2" thru_hole circle
 			(at 14.38 31 270)
-			(size 2.286 2.286)
-			(drill 1.27)
+			(size 2.8 2.8)
+			(drill 1.5)
 			(layers "*.Cu" "*.Mask")
 			(remove_unused_layers no)
@@
 		(pad "3" thru_hole circle
 			(at 20.73 31 270)
-			(size 2.286 2.286)
-			(drill 1.27)
+			(size 2.8 2.8)
+			(drill 1.5)
 			(layers "*.Cu" "*.Mask")
 			(remove_unused_layers no)
@@
 		(pad "4" thru_hole circle
 			(at 27.07 31 270)
-			(size 2.286 2.286)
-			(drill 1.27)
+			(size 2.8 2.8)
+			(drill 1.5)
 			(layers "*.Cu" "*.Mask")
 			(remove_unused_layers no)
@@
 		(pad "5" thru_hole circle
 			(at 8.03 0 270)
-			(size 2.286 2.286)
-			(drill 1.27)
+			(size 2.8 2.8)
+			(drill 1.5)
 			(layers "*.Cu" "*.Mask")
 			(remove_unused_layers no)
@@
 		(pad "6" thru_hole circle
 			(at 14.38 0 270)
-			(size 2.286 2.286)
-			(drill 1.27)
+			(size 2.8 2.8)
+			(drill 1.5)
 			(layers "*.Cu" "*.Mask")
 			(remove_unused_layers no)
@@
 		(pad "7" thru_hole circle
 			(at 20.73 0 270)
-			(size 2.286 2.286)
-			(drill 1.27)
+			(size 2.8 2.8)
+			(drill 1.5)
 			(layers "*.Cu" "*.Mask")
 			(remove_unused_layers no)
@@
 		(pad "8" thru_hole circle
 			(at 27.07 0 270)
-			(size 2.286 2.286)
-			(drill 1.27)
+			(size 2.8 2.8)
+			(drill 1.5)
 			(layers "*.Cu" "*.Mask")
 			(remove_unused_layers no)
@@
 	(footprint "Symbol:Symbol_HighVoltage_Type2_CopperTop_VerySmall"
 		(layer "F.Cu")
-		(at 71.12 110.49)
+		(at 70.95 108.85)
 		(descr "Symbol, High Voltage, Type 2, Copper Top, Very Small,")
 		(tags "Symbol, High Voltage, Type 2, Copper Top, Very Small,")
@@
 	)
 	(segment
-		(start 96.9065 178.6885)
-		(end 59.3085 178.6885)
+		(start 59.3085 178.6885)
+		(end 58.42 177.8)
 		(width 0.25)
 		(layer "F.Cu")
@@
 	)
 	(segment
-		(start 59.3085 178.6885)
-		(end 58.42 177.8)
+		(start 98.6 177.8)
+		(end 98.7 177.7)
 		(width 0.25)
-		(layer "F.Cu")
+		(layer "B.Cu")
 		(net 5)
 	)
 	(segment
-		(start 96.5883 108.649)
-		(end 58.991 108.649)
+		(start 58.42 109.22)
+		(end 97.97 109.22)
 		(width 0.25)
-		(layer "F.Cu")
+		(layer "B.Cu")
+		(net 5)
+	)
+	(segment
+		(start 97.97 109.22)
+		(end 98 109.25)
+		(width 0.25)
+		(layer "B.Cu")
+		(net 5)
+	)
+	(segment
+		(start 58.42 177.8)
+		(end 98.6 177.8)
+		(width 0.25)
+		(layer "B.Cu")
 		(net 5)
 	)
@@
 	)
 	(segment
-		(start 110.49 119.38)
+		(start 114.915 119.135)
 		(end 110.49 114.71)
 		(width 0.25)
@@
 	)
 	(segment
+		(start 114.915 123.805)
+		(end 114.915 119.135)
+		(width 0.25)
+		(layer "F.Cu")
+		(net 28)
+	)
+	(segment
 		(start 116.84 125.73)
-		(end 110.49 119.38)
+		(end 114.915 123.805)
 		(width 0.25)
 		(layer "F.Cu")
@@
 	)
 	(segment
-		(start 116.84 162.56)
-		(end 110.003 169.397)
+		(start 110.003 169.397)
+		(end 116.84 162.56)
 		(width 0.25)
 		(layer "B.Cu")
@@
 	)
 	(segment
-		(start 110.003 169.397)
-		(end 110.003 172.945)
+		(start 110.003 172.945)
+		(end 110.003 169.397)
 		(width 0.25)
 		(layer "B.Cu")
@@
 		(net 5)
 		(net_name "GND")
-		(layer "F.Cu")
-		(hatch edge 0.508)
-		(connect_pads
-			(clearance 0.508)
-		)
-		(min_thickness 0.254)
-		(filled_areas_thickness no)
-		(fill yes
-			(thermal_gap 0.508)
-			(thermal_bridge_width 0.508)
-		)
-		(polygon
-			(pts
-				(xy 147.574 181.61) (xy 95.25 181.61) (xy 95.25 105.41) (xy 147.574 105.41)
-			)
-		)
-	)
-	(zone
-		(net 5)
-		(net_name "GND")
-		(layer "B.Cu")
+		(layers "F&B.Cu")
 		(hatch edge 0.508)
 		(connect_pads
