File: VoltageMeter/VoltageMeter.kicad_sch (KiCad schematic)
At the start: 17 parts, among them J1 Conn_01x02_Male, J2 Conn_01x02_Male

Commit message: A few updates to clean things up.
Parts:
- D3, D4: value D_Zener -> 5V
- R1, R2: symbol Device:R -> Device:R_US
- R3, R4: symbol Device:R_Small -> Device:R_US
- RV1, RV2: symbol VoltageMeter-rescue:R_POT_TRIM-Device -> Device:R_Potentiometer_US
Changed lines of the file:
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@@
 	)
 	(symbol
-		(lib_id "VoltageMeter-rescue:R_POT_TRIM-Device")
+		(lib_id "Device:R_Potentiometer_US")
 		(at 124.46 62.23 90)
 		(mirror x)
@@
 			)
 		)
-		(property "Description" ""
+		(property "Description" "Potentiometer, US symbol"
 			(at 124.46 62.23 0)
 			(effects
@@
 	)
 	(symbol
-		(lib_id "Device:R_Small")
-		(at 124.46 39.37 0)
+		(lib_id "Device:R_US")
+		(at 124.46 40.64 0)
 		(unit 1)
 		(exclude_from_sim no)
@@
 		(dnp no)
 		(property "Reference" "R3"
-			(at 125.9586 38.2016 0)
+			(at 125.9586 39.4716 0)
 			(effects
 				(font
@@
 		)
 		(property "Value" "120k"
-			(at 125.9586 40.513 0)
+			(at 125.9586 41.783 0)
 			(effects
 				(font
@@
 		)
 		(property "Footprint" "Resistor_THT:R_Axial_DIN0207_L6.3mm_D2.5mm_P10.16mm_Horizontal"
-			(at 124.46 39.37 0)
-			(effects
-				(font
-					(size 1.27 1.27)
-				)
-				(hide yes)
-			)
-		)
-		(property "Datasheet" "~"
-			(at 124.46 39.37 0)
-			(effects
-				(font
-					(size 1.27 1.27)
-				)
-				(hide yes)
-			)
-		)
-		(property "Description" ""
-			(at 124.46 39.37 0)
+			(at 125.476 40.894 90)
+			(effects
+				(font
+					(size 1.27 1.27)
+				)
+				(hide yes)
+			)
+		)
+		(property "Datasheet" "~"
+			(at 124.46 40.64 0)
+			(effects
+				(font
+					(size 1.27 1.27)
+				)
+				(hide yes)
+			)
+		)
+		(property "Description" "Resistor, US symbol"
+			(at 124.46 40.64 0)
 			(effects
 				(font
@@
 	)
 	(symbol
-		(lib_id "VoltageMeter-rescue:R_POT_TRIM-Device")
+		(lib_id "Device:R_Potentiometer_US")
 		(at 124.46 29.21 90)
 		(mirror x)
@@
 			)
 		)
-		(property "Description" ""
+		(property "Description" "Potentiometer, US symbol"
 			(at 124.46 29.21 0)
 			(effects
@@
 	)
 	(symbol
-		(lib_id "Device:R_Small")
-		(at 124.46 72.39 0)
+		(lib_id "Device:R_US")
+		(at 124.46 73.66 0)
 		(unit 1)
 		(exclude_from_sim no)
@@
 		(dnp no)
 		(property "Reference" "R4"
-			(at 125.9586 71.2216 0)
+			(at 125.9586 72.4916 0)
 			(effects
 				(font
@@
 		)
 		(property "Value" "120k"
-			(at 125.9586 73.533 0)
+			(at 125.9586 74.803 0)
 			(effects
 				(font
@@
 		)
 		(property "Footprint" "Resistor_THT:R_Axial_DIN0207_L6.3mm_D2.5mm_P10.16mm_Horizontal"
-			(at 124.46 72.39 0)
-			(effects
-				(font
-					(size 1.27 1.27)
-				)
-				(hide yes)
-			)
-		)
-		(property "Datasheet" "~"
-			(at 124.46 72.39 0)
-			(effects
-				(font
-					(size 1.27 1.27)
-				)
-				(hide yes)
-			)
-		)
-		(property "Description" ""
-			(at 124.46 72.39 0)
+			(at 125.476 73.914 90)
+			(effects
+				(font
+					(size 1.27 1.27)
+				)
+				(hide yes)
+			)
+		)
+		(property "Datasheet" "~"
+			(at 124.46 73.66 0)
+			(effects
+				(font
+					(size 1.27 1.27)
+				)
+				(hide yes)
+			)
+		)
+		(property "Description" "Resistor, US symbol"
+			(at 124.46 73.66 0)
 			(effects
 				(font
@@
 	)
 	(symbol
-		(lib_id "Device:R")
+		(lib_id "Device:R_US")
 		(at 116.84 29.21 270)
 		(unit 1)
@@
 		)
 		(property "Footprint" "Resistor_THT:R_Axial_DIN0207_L6.3mm_D2.5mm_P10.16mm_Horizontal"
-			(at 116.84 27.432 90)
+			(at 116.586 30.226 90)
 			(effects
 				(font
@@
 			)
 		)
-		(property "Description" ""
+		(property "Description" "Resistor, US symbol"
 			(at 116.84 29.21 0)
 			(effects
@@
 	)
 	(symbol
-		(lib_id "Device:R")
+		(lib_id "Device:R_US")
 		(at 116.84 62.23 270)
 		(unit 1)
@@
 		)
 		(property "Footprint" "Resistor_THT:R_Axial_DIN0207_L6.3mm_D2.5mm_P10.16mm_Horizontal"
-			(at 116.84 60.452 90)
+			(at 116.586 63.246 90)
 			(effects
 				(font
@@
 			)
 		)
-		(property "Description" ""
+		(property "Description" "Resistor, US symbol"
 			(at 116.84 62.23 0)
 			(effects
@@
 			)
 		)
-		(property "Value" "D_Zener"
+		(property "Value" "5V"
 			(at 134.112 39.243 90)
 			(effects
@@
 			)
 		)
-		(property "Value" "D_Zener"
+		(property "Value" "5V"
 			(at 134.112 72.263 90)
 			(effects
@@
 	(symbol
 		(lib_id "VoltageMeter-rescue:GND-power")
-		(at 124.46 41.91 0)
+		(at 124.46 44.45 0)
 		(unit 1)
 		(exclude_from_sim no)
@@
 		(dnp no)
 		(property "Reference" "#PWR02"
-			(at 124.46 48.26 0)
+			(at 124.46 50.8 0)
 			(effects
 				(font
@@
 		)
 		(property "Value" "GND"
-			(at 124.587 46.3042 0)
+			(at 124.587 48.8442 0)
 			(effects
 				(font
@@
 		)
 		(property "Footprint" ""
-			(at 124.46 41.91 0)
+			(at 124.46 44.45 0)
 			(effects
 				(font
@@
 		)
 		(property "Datasheet" ""
-			(at 124.46 41.91 0)
+			(at 124.46 44.45 0)
 			(effects
 				(font
@@
 		)
 		(property "Description" ""
-			(at 124.46 41.91 0)
+			(at 124.46 44.45 0)
 			(effects
 				(font
@@
 	(symbol
 		(lib_id "VoltageMeter-rescue:GND-power")
-		(at 124.46 74.93 0)
+		(at 124.46 77.47 0)
 		(unit 1)
 		(exclude_from_sim no)
@@
 		(dnp no)
 		(property "Reference" "#PWR05"
-			(at 124.46 81.28 0)
+			(at 124.46 83.82 0)
 			(effects
 				(font
@@
 		)
 		(property "Value" "GND"
-			(at 124.587 79.3242 0)
+			(at 124.587 81.8642 0)
 			(effects
 				(font
@@
 		)
 		(property "Footprint" ""
-			(at 124.46 74.93 0)
+			(at 124.46 77.47 0)
 			(effects
 				(font
@@
 		)
 		(property "Datasheet" ""
-			(at 124.46 74.93 0)
+			(at 124.46 77.47 0)
 			(effects
 				(font
@@
 		)
 		(property "Description" ""
-			(at 124.46 74.93 0)
-			(effects
-				(font
+			(at 124.46 77.47 0)
+			(effects
+				(font
